File: justanultrasonicthingy/justanultrasonicthingy.kicad_sch (KiCad schematic)
At the start: 0 parts

Commit message: Wired the simple ultrasonic sensor to the xiao board
Parts:
- added BT1: Battery, symbol Device:Battery
- added DS1: WC1602A, Display:WC1602A, symbol Display_Character:WC1602A
- added SW1: SW_Push, symbol Switch:SW_Push
- added U1: XIAO-RP2040-DIP, Module:MOUDLE14P-XIAO-DIP-SMD, symbol Seeed_Studio_XIAO_Series:XIAO-RP2040-DIP
- added U2: HC-SR04, HC-SR04:XCVR_HC-SR04, symbol HC-SR04:HC-SR04
- added U3: PCF8574AP, Package_DIP:DIP-16_W7.62mm, symbol Interface_Expansion:PCF8574AP
Connections:
- new net: BT1.1 (+), SW1.1
- new net: DS1.12 (D5), U3.10 (P5)
- new net: DS1.13 (D6), U3.11 (P6)
- new net: DS1.14 (D7), U3.12 (P7)
- new net: DS1.7 (D0), U3.4 (P0)
- new net: DS1.8 (D1), U3.5 (P1)
- new net: DS1.9 (D2), U3.6 (P2)
- new net: DS1.10 (D3), U3.7 (P3)
- new net: DS1.11 (D4), U3.9 (P4)
- new net GND: BT1.2 (-), U1.13 (GND), U2.4 (GND)
- new net echo: U1.3 (GPIO28/ADC2/A2), U2.3 (ECHO)
- new net powah: SW1.2, U1.14 (VBUS), U2.1 (VCC)
- new net trig: U1.2 (GPIO27/ADC1/A1), U2.2 (TRIG)

Commit message: Added 4 pin holes for the display stuff and two pin holes for the battery
Parts:
- removed DS1: WC1602A, Display:WC1602A, symbol Display_Character:WC1602A
- removed U3: PCF8574AP, Package_DIP:DIP-16_W7.62mm, symbol Interface_Expansion:PCF8574AP
- added Displaystuff1: Conn_01x04_Pin, Connector:FanPinHeader_1x04_P2.54mm_Vertical, symbol Connector:Conn_01x04_Pin
- BT1: footprint (none) -> Connector_PinHeader_2.54mm:PinHeader_1x02_P2.54mm_Vertical
- SW1: footprint (none) -> Button_Switch_THT:SW_PUSH_6mm
Connections:
- net GND: now also Displaystuff1.4 (Pin_4)
- net powah: now also Displaystuff1.3 (Pin_3)
- net SDA: now reaches U1.5 (GPIO6/SDA)
- net SDA: now also Displaystuff1.2 (Pin_2)
- net SCL: now reaches U1.6 (GPIO7/SCL)
- net SCL: now also Displaystuff1.1 (Pin_1)

Commit message: Added all the stuff with a few workarounds
Parts:
- Displaystuff1: footprint Connector:FanPinHeader_1x04_P2.54mm_Vertical -> Connector_PinHeader_2.54mm:PinHeader_1x04_P2.54mm_Vertical
- U1: footprint Module:MOUDLE14P-XIAO-DIP-SMD -> footprints:XIAO-RP2040-DIP
- U2: footprint HC-SR04:XCVR_HC-SR04 -> HC-SR04 FOOTPRINT:XCVR_HC-SR04
Changed lines of the file:
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@@
 			)
 		)
-		(property "Footprint" "Connector:FanPinHeader_1x04_P2.54mm_Vertical"
+		(property "Footprint" "Connector_PinHeader_2.54mm:PinHeader_1x04_P2.54mm_Vertical"
 			(at 77.47 82.55 0)
 			(effects
@@
 			)
 		)
-		(property "Footprint" "Module:MOUDLE14P-XIAO-DIP-SMD"
+		(property "Footprint" "footprints:XIAO-RP2040-DIP"
 			(at 90.678 74.168 0)
 			(effects
@@
 			)
 		)
-		(property "Footprint" "HC-SR04:XCVR_HC-SR04"
+		(property "Footprint" "HC-SR04 FOOTPRINT:XCVR_HC-SR04"
 			(at 119.38 30.48 0)
 			(effects

Commit message: Added Resistors for the components
Parts:
- added R1, R2: R, symbol Device:R
Connections:
- net powah: now also R1.1, R2.1; no longer Displaystuff1.3 (Pin_3), U2.1 (VCC)
- new net: Displaystuff1.3 (Pin_3), R2.2
- new net: R1.2, U2.1 (VCC)
Changed lines of the file:
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@@
+	(wire
+		(pts
+			(xy 43.18 77.47) (xy 72.39 77.47)
+		)
+		(stroke
+			(width 0)
+			(type default)
+		)
+	)
 	(wire
 		(pts
@@
 	(wire
 		(pts
-			(xy 72.39 77.47) (xy 55.88 77.47)
+			(xy 43.18 77.47) (xy 43.18 78.74)
 		)
 		(stroke
@@
 		)
 	)
-	(wire
-		(pts
-			(xy 55.88 77.47) (xy 55.88 78.74)
-		)
-		(stroke
-			(width 0)
-			(type default)
-		)
-	)
 	(global_label "SDA"
 		(shape input)
@@
 	(global_label "powah"
 		(shape input)
-		(at 72.39 80.01 180)
+		(at 64.77 80.01 180)
 		(fields_autoplaced yes)
 		(effects
@@
 		)
 		(property "Intersheetrefs" "${INTERSHEET_REFS}"
-			(at 63.4783 80.01 0)
+			(at 55.8583 80.01 0)
 			(effects
 				(font
@@
 	(global_label "powah"
 		(shape input)
-		(at 114.3 27.94 180)
+		(at 106.68 27.94 180)
 		(fields_autoplaced yes)
 		(effects
@@
 		)
 		(property "Intersheetrefs" "${INTERSHEET_REFS}"
-			(at 105.3883 27.94 0)
+			(at 97.7683 27.94 0)
 			(effects
 				(font
@@
 	)
 	(symbol
+		(lib_id "Device:R")
+		(at 68.58 80.01 90)
+		(unit 1)
+		(exclude_from_sim no)
+		(in_bom yes)
+		(on_board yes)
+		(dnp no)
+		(fields_autoplaced yes)
+		(property "Reference" "R2"
+			(at 68.58 73.66 90)
+			(effects
+				(font
+					(size 1.27 1.27)
+				)
+			)
+		)
+		(property "Value" "R"
+			(at 68.58 76.2 90)
+			(effects
+				(font
+					(size 1.27 1.27)
+				)
+			)
+		)
+		(property "Footprint" ""
+			(at 68.58 81.788 90)
+			(effects
+				(font
+					(size 1.27 1.27)
+				)
+				(hide yes)
+			)
+		)
+		(property "Datasheet" "~"
+			(at 68.58 80.01 0)
+			(effects
+				(font
+					(size 1.27 1.27)
+				)
+				(hide yes)
+			)
+		)
+		(property "Description" "Resistor"
+			(at 68.58 80.01 0)
+			(effects
+				(font
+					(size 1.27 1.27)
+				)
+				(hide yes)
+			)
+		)
+		(pin "1"
+		)
+		(pin "2"
+		)
+		(instances
+			(project "justanultrasonicthingy"
+				(path "/f211ce28-fabb-437c-ba0f-1b91711cc7e9"
+					(reference "R2")
+					(unit 1)
+				)
+			)
+		)
+	)
+	(symbol
 		(lib_id "Switch:SW_Push")
 		(at 64.77 30.48 0)
@@
 	)
 	(symbol
-		(lib_id "power:GND")
-		(at 55.88 78.74 0)
+		(lib_id "Device:R")
+		(at 110.49 27.94 90)
 		(unit 1)
 		(exclude_from_sim no)
@@
 		(dnp no)
 		(fields_autoplaced yes)
+		(property "Reference" "R1"
+			(at 110.49 21.59 90)
+			(effects
+				(font
+					(size 1.27 1.27)
+				)
+			)
+		)
+		(property "Value" "R"
+			(at 110.49 24.13 90)
+			(effects
+				(font
+					(size 1.27 1.27)
+				)
+			)
+		)
+		(property "Footprint" ""
+			(at 110.49 29.718 90)
+			(effects
+				(font
+					(size 1.27 1.27)
+				)
+				(hide yes)
+			)
+		)
+		(property "Datasheet" "~"
+			(at 110.49 27.94 0)
+			(effects
+				(font
+					(size 1.27 1.27)
+				)
+				(hide yes)
+			)
+		)
+		(property "Description" "Resistor"
+			(at 110.49 27.94 0)
+			(effects
+				(font
+					(size 1.27 1.27)
+				)
+				(hide yes)
+			)
+		)
+		(pin "1"
+		)
+		(pin "2"
+		)
+		(instances
+			(project ""
+				(path "/f211ce28-fabb-437c-ba0f-1b91711cc7e9"
+					(reference "R1")
+					(unit 1)
+				)
+			)
+		)
+	)
+	(symbol
+		(lib_id "power:GND")
+		(at 43.18 78.74 0)
+		(unit 1)
+		(exclude_from_sim no)
+		(in_bom yes)
+		(on_board yes)
+		(dnp no)
+		(fields_autoplaced yes)
 		(property "Reference" "#PWR04"
-			(at 55.88 85.09 0)
+			(at 43.18 85.09 0)
 			(effects
 				(font
@@
 		)
 		(property "Value" "GND"
-			(at 55.88 83.82 0)
+			(at 43.18 83.82 0)
 			(effects
 				(font
@@
 		)
 		(property "Footprint" ""
-			(at 55.88 78.74 0)
+			(at 43.18 78.74 0)
 			(effects
 				(font
@@
 		)
 		(property "Datasheet" ""
-			(at 55.88 78.74 0)
+			(at 43.18 78.74 0)
 			(effects
 				(font
@@
 		)
 		(property "Description" "Power symbol creates a global label with name \"GND\" , ground"
-			(at 55.88 78.74 0)
-			(effects
-				(font
+			(at 43.18 78.74 0)
+			(effects
+				(font

Commit message: Added a small led indicator for the pcb when it is turned on
Parts:
- added D1: LED, symbol Device:LED
- added R3: R, symbol Device:R
Connections:
- net GND: now also D1.1 (K)
- net powah: now also R3.2
- new net: D1.2 (A), R3.1
Changed lines of the file:
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@@
+	(global_label "powah"
+		(shape input)
+		(at 138.43 45.72 180)
+		(fields_autoplaced yes)
+		(effects
+			(font
+				(size 1.27 1.27)
+			)
+			(justify right)
+		)
+		(property "Intersheetrefs" "${INTERSHEET_REFS}"
+			(at 129.5183 45.72 0)
+			(effects
+				(font
+					(size 1.27 1.27)
+				)
+				(justify right)
+				(hide yes)
+			)
+		)
+	)
 	(global_label "powah"
 		(shape input)
@@
 	)
 	(symbol
+		(lib_id "Device:LED")
+		(at 149.86 45.72 180)
+		(unit 1)
+		(exclude_from_sim no)
+		(in_bom yes)
+		(on_board yes)
+		(dnp no)
+		(fields_autoplaced yes)
+		(property "Reference" "D1"
+			(at 151.4475 38.1 0)
+			(effects
+				(font
+					(size 1.27 1.27)
+				)
+			)
+		)
+		(property "Value" "LED"
+			(at 151.4475 40.64 0)
+			(effects
+				(font
+					(size 1.27 1.27)
+				)
+			)
+		)
+		(property "Footprint" ""
+			(at 149.86 45.72 0)
+			(effects
+				(font
+					(size 1.27 1.27)
+				)
+				(hide yes)
+			)
+		)
+		(property "Datasheet" "~"
+			(at 149.86 45.72 0)
+			(effects
+				(font
+					(size 1.27 1.27)
+				)
+				(hide yes)
+			)
+		)
+		(property "Description" "Light emitting diode"
+			(at 149.86 45.72 0)
+			(effects
+				(font
+					(size 1.27 1.27)
+				)
+				(hide yes)
+			)
+		)
+		(property "Sim.Pins" "1=K 2=A"
+			(at 149.86 45.72 0)
+			(effects
+				(font
+					(size 1.27 1.27)
+				)
+				(hide yes)
+			)
+		)
+		(pin "1"
+		)
+		(pin "2"
+		)
+		(instances
+			(project ""
+				(path "/f211ce28-fabb-437c-ba0f-1b91711cc7e9"
+					(reference "D1")
+					(unit 1)
+				)
+			)
+		)
+	)
+	(symbol
 		(lib_id "Switch:SW_Push")
 		(at 64.77 30.48 0)
@@
 					(unit 1)
 				)
+			)
+		)
+	)
+	(symbol
+		(lib_id "Device:R")
+		(at 142.24 45.72 270)
+		(unit 1)
+		(exclude_from_sim no)
+		(in_bom yes)
+		(on_board yes)
+		(dnp no)
+		(fields_autoplaced yes)
+		(property "Reference" "R3"
+			(at 142.24 39.37 90)
+			(effects
+				(font
+					(size 1.27 1.27)
+				)
+			)
+		)
+		(property "Value" "R"
+			(at 142.24 41.91 90)
+			(effects
+				(font
+					(size 1.27 1.27)
+				)
+			)
+		)
+		(property "Footprint" ""
+			(at 142.24 43.942 90)
+			(effects
+				(font
+					(size 1.27 1.27)
+				)
+				(hide yes)
+			)
+		)
+		(property "Datasheet" "~"
+			(at 142.24 45.72 0)
+			(effects
+				(font
+					(size 1.27 1.27)
+				)
+				(hide yes)
+			)
+		)
+		(property "Description" "Resistor"
+			(at 142.24 45.72 0)
+			(effects
+				(font
+					(size 1.27 1.27)
+				)
+				(hide yes)
+			)
+		)
+		(pin "1"
+		)
+		(pin "2"
+		)
+		(instances
+			(project ""
+				(path "/f211ce28-fabb-437c-ba0f-1b91711cc7e9"
+					(reference "R3")
+					(unit 1)
+				)
+			)
+		)
+	)
+	(symbol
+		(lib_id "power:GND")
+		(at 153.67 45.72 0)
+		(unit 1)
+		(exclude_from_sim no)
+		(in_bom yes)
+		(on_board yes)
+		(dnp no)
+		(fields_autoplaced yes)
+		(property "Reference" "#PWR05"
+			(at 153.67 52.07 0)
+			(effects
+				(font
+					(size 1.27 1.27)
+				)
+				(hide yes)
+			)
+		)
+		(property "Value" "GND"
+			(at 153.67 50.8 0)
+			(effects
+				(font
+					(size 1.27 1.27)
+				)
+			)
+		)
+		(property "Footprint" ""
+			(at 153.67 45.72 0)
+			(effects
+				(font
+					(size 1.27 1.27)
+				)
+				(hide yes)
+			)
+		)
+		(property "Datasheet" ""
+			(at 153.67 45.72 0)
+			(effects
+				(font
+					(size 1.27 1.27)
+				)
+				(hide yes)
+			)
+		)
+		(property "Description" "Power symbol creates a global label with name \"GND\" , ground"
+			(at 153.67 45.72 0)
+			(effects
+				(font
+					(size 1.27 1.27)
+				)
+				(hide yes)
+			)
+		)
+		(pin "1"
+		)
+		(instances
+			(project ""
+				(path "/f211ce28-fabb-437c-ba0f-1b91711cc7e9"
+					(reference "#PWR05")
+					(unit 1)
+				)

Commit message: Added the laser stuff in the pcb
Parts:
- added D2: LASER, Connector_PinHeader_2.54mm:PinHeader_1x02_P2.54mm_Vertical, symbol Device:LED
- added R4: R, Resistor_THT:R_Axial_DIN0207_L6.3mm_D2.5mm_P7.62mm_Horizontal, symbol Device:R
- D1: footprint (none) -> LED_THT:LED_D5.0mm
- R1, R2, R3: footprint (none) -> Resistor_THT:R_Axial_DIN0207_L6.3mm_D2.5mm_P7.62mm_Horizontal
Connections:
- net GND: now also D2.1 (K)
- net powah: now also R4.2
- new net: D2.2 (A), R4.1
Changed lines of the file:
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@@
+		)
+	)
+	(global_label "powah"
+		(shape input)
+		(at 140.97 63.5 180)
+		(fields_autoplaced yes)
+		(effects
+			(font
+				(size 1.27 1.27)
+			)
+			(justify right)
+		)
+		(property "Intersheetrefs" "${INTERSHEET_REFS}"
+			(at 132.0583 63.5 0)
+			(effects
+				(font
+					(size 1.27 1.27)
+				)
+				(justify right)
+				(hide yes)
+			)
+		)
+		(property "Netclass" ""
+			(at 140.97 65.6908 0)
+			(effects
+				(font
+					(size 1.27 1.27)
+				)
+				(justify right)
+				(hide yes)
+			)
 		)
 	)
@@
 			)
 		)
-		(property "Footprint" ""
+		(property "Footprint" "Resistor_THT:R_Axial_DIN0207_L6.3mm_D2.5mm_P7.62mm_Horizontal"
 			(at 68.58 81.788 90)
 			(effects
@@
 	)
 	(symbol
+		(lib_id "power:GND")
+		(at 156.21 63.5 0)
+		(unit 1)
+		(exclude_from_sim no)
+		(in_bom yes)
+		(on_board yes)
+		(dnp no)
+		(fields_autoplaced yes)
+		(property "Reference" "#PWR06"
+			(at 156.21 69.85 0)
+			(effects
+				(font
+					(size 1.27 1.27)
+				)
+				(hide yes)
+			)
+		)
+		(property "Value" "GND"
+			(at 156.21 68.58 0)
+			(effects
+				(font
+					(size 1.27 1.27)
+				)
+			)
+		)
+		(property "Footprint" ""
+			(at 156.21 63.5 0)
+			(effects
+				(font
+					(size 1.27 1.27)
+				)
+				(hide yes)
+			)
+		)
+		(property "Datasheet" ""
+			(at 156.21 63.5 0)
+			(effects
+				(font
+					(size 1.27 1.27)
+				)
+				(hide yes)
+			)
+		)
+		(property "Description" "Power symbol creates a global label with name \"GND\" , ground"
+			(at 156.21 63.5 0)
+			(effects
+				(font
+					(size 1.27 1.27)
+				)
+				(hide yes)
+			)
+		)
+		(pin "1"
+		)
+		(instances
+			(project "justanultrasonicthingy"
+				(path "/f211ce28-fabb-437c-ba0f-1b91711cc7e9"
+					(reference "#PWR06")
+					(unit 1)
+				)
+			)
+		)
+	)
+	(symbol
+		(lib_id "Device:R")
+		(at 144.78 63.5 270)
+		(unit 1)
+		(exclude_from_sim no)
+		(in_bom yes)
+		(on_board yes)
+		(dnp no)
+		(fields_autoplaced yes)
+		(property "Reference" "R4"
+			(at 144.78 57.15 90)
+			(effects
+				(font
+					(size 1.27 1.27)
+				)
+			)
+		)
+		(property "Value" "R"
+			(at 144.78 59.69 90)
+			(effects
+				(font
+					(size 1.27 1.27)
+				)
+			)
+		)
+		(property "Footprint" "Resistor_THT:R_Axial_DIN0207_L6.3mm_D2.5mm_P7.62mm_Horizontal"
+			(at 144.78 61.722 90)
+			(effects
+				(font
+					(size 1.27 1.27)
+				)
+				(hide yes)
+			)
+		)
+		(property "Datasheet" "~"
+			(at 144.78 63.5 0)
+			(effects
+				(font
+					(size 1.27 1.27)
+				)
+				(hide yes)
+			)
+		)
+		(property "Description" "Resistor"
+			(at 144.78 63.5 0)
+			(effects
+				(font
+					(size 1.27 1.27)
+				)
+				(hide yes)
+			)
+		)
+		(pin "1"
+		)
+		(pin "2"
+		)
+		(instances
+			(project "justanultrasonicthingy"
+				(path "/f211ce28-fabb-437c-ba0f-1b91711cc7e9"
+					(reference "R4")
+					(unit 1)
+				)
+			)
+		)
+	)
+	(symbol
 		(lib_id "Device:LED")
 		(at 149.86 45.72 180)
@@
 			)
 		)
-		(property "Footprint" ""
+		(property "Footprint" "LED_THT:LED_D5.0mm"
 			(at 149.86 45.72 0)
 			(effects
@@
 			)
 		)
-		(property "Footprint" ""
+		(property "Footprint" "Resistor_THT:R_Axial_DIN0207_L6.3mm_D2.5mm_P7.62mm_Horizontal"
 			(at 142.24 43.942 90)
 			(effects
@@
 	)
 	(symbol
+		(lib_id "Device:LED")
+		(at 152.4 63.5 180)
+		(unit 1)
+		(exclude_from_sim no)
+		(in_bom yes)
+		(on_board yes)
+		(dnp no)
+		(fields_autoplaced yes)
+		(property "Reference" "D2"
+			(at 153.9875 55.88 0)
+			(effects
+				(font
+					(size 1.27 1.27)
+				)
+			)
+		)
+		(property "Value" "LASER"
+			(at 153.9875 58.42 0)
+			(effects
+				(font
+					(size 1.27 1.27)
+				)
+			)
+		)
+		(property "Footprint" "Connector_PinHeader_2.54mm:PinHeader_1x02_P2.54mm_Vertical"
+			(at 152.4 63.5 0)
+			(effects
+				(font
+					(size 1.27 1.27)
+				)
+				(hide yes)
+			)
+		)
+		(property "Datasheet" "~"
+			(at 152.4 63.5 0)
+			(effects
+				(font
+					(size 1.27 1.27)
+				)
+				(hide yes)
+			)
+		)
+		(property "Description" "Light emitting diode"
+			(at 152.4 63.5 0)
+			(effects
+				(font
+					(size 1.27 1.27)
+				)
+				(hide yes)
+			)
+		)
+		(property "Sim.Pins" "1=K 2=A"
+			(at 152.4 63.5 0)
+			(effects
+				(font
+					(size 1.27 1.27)
+				)
+				(hide yes)
+			)
+		)
+		(pin "1"
+		)
+		(pin "2"
+		)
+		(instances
+			(project "justanultrasonicthingy"
+				(path "/f211ce28-fabb-437c-ba0f-1b91711cc7e9"
+					(reference "D2")
+					(unit 1)
+				)
+			)
+		)
+	)
+	(symbol
 		(lib_id "HC-SR04:HC-SR04")
 		(at 119.38 30.48 0)
@@
 			)
 		)
-		(property "Footprint" ""
+		(property "Footprint" "Resistor_THT:R_Axial_DIN0207_L6.3mm_D2.5mm_P7.62mm_Horizontal"
 			(at 110.49 29.718 90)
 			(effects
